Commit message: Update drone racing tasks, track, and control setup

File: resources/models/environment_assets/racing/cylinder_obstacle.urdf (robot description, URDF)
Before this commit: robot cylinder_obstacle, 1 links, 0 joints
Links:
- link base_link: geometry collision cylinder length=4.5 radius=0.20; visual cylinder length=4.5 radius=0.20

File: resources/models/environment_assets/racing/gate_1p5m.urdf (robot description, URDF)
Before this commit: robot race_gate_1p5m, 5 links, 4 joints
Links:
- link bottom_bar: geometry collision box size=0.45 4.64 0.32; visual box size=0.45 4.64 0.32
- link left_bar: geometry collision box size=0.45 0.32 4.64; visual box size=0.45 0.32 4.64
- link right_bar: geometry collision box size=0.45 0.32 4.64; visual box size=0.45 0.32 4.64
- link top_bar: geometry collision box size=0.45 4.64 0.32; visual box size=0.45 4.64 0.32
Joints:
- joint base_to_bottom_bar: origin xyz=0 0 -1.125 rpy=0 0 0 -> xyz=0 0 -2.16 rpy=0 0 0
- joint base_to_left_bar: origin xyz=0 1.125 0 rpy=0 0 0 -> xyz=0 2.16 0 rpy=0 0 0
- joint base_to_right_bar: origin xyz=0 -1.125 0 rpy=0 0 0 -> xyz=0 -2.16 0 rpy=0 0 0
- joint base_to_top_bar: origin xyz=0 0 1.125 rpy=0 0 0 -> xyz=0 0 2.16 rpy=0 0 0

Commit message: success and more entities

File: resources/models/environment_assets/racing/cylinder_obstacle.urdf (robot description, URDF)
Before this commit: robot cylinder_obstacle, 1 links, 0 joints
Links:
- link base_link: geometry collision cylinder length=9.0 radius=0.55; visual cylinder length=9.0 radius=0.55
